Commit message: WIP adding xacro

File: models/Omniveyor/omniveyor.gazebo.xacro (robot description, xacro)
@@ -1,11 +1,6 @@
-<?xml version='1.0'?>
-<sdf version='1.6'>
-  <model name="omniveyor_robot">
-    <!-- For debug purpose Only: When configuring the robot structure,
-         setting static to true such that the robot is ignored by the physics engine.
-      -->
-    <!--static>true</static-->
-    <!-- Robot base_link -->
-    <link name='base_link'>
+<?xml version="1.0" ?>
+<robot name="omniveyor" xmlns:xacro="http://www.ros.org/wiki/xacro">
+  <!-- Robot base_link -->
+  <gazebo reference="base_link">
       <pose>0 0 0 0 0 0</pose>
       <inertial>
@@ -30,11 +25,4 @@
         <pose>-0.3752 0.3381 0.032 1.5708 -0 0</pose>
       </collision>
-      <!--visual name='visual'>
-        <geometry>
-          <box>
-            <size>0.62 0.62 0.32</size>
-          </box>
-        </geometry>
-      </visual-->
       <visual name='visual_mesh'>
         <geometry>
@@ -52,5 +40,6 @@
         </material>
       </visual>
-    </link>
+  </gazebo>
+  <gazebo>
     <!-- Powered Casters -->
     <link name="FL_wheel">
@@ -383,252 +372,4 @@
         </geometry>
       </visual>
-    </link>
-    <link name="hokuyo">
-      <pose>0.27 0 0.08 0 0 0</pose>
-      <inertial>
-        <mass>0.1</mass>
-        <inertia>
-          <ixx>0.01</ixx>
-          <ixy>0</ixy>
-          <ixz>0</ixz>
-          <iyy>0.01</iyy>
-          <iyz>0</iyz>
-          <izz>0.01</izz>
-        </inertia>
-      </inertial>
-      <visual name="visual">
-        <geometry>
-          <mesh>
-            <uri>model://hokuyo/meshes/hokuyo.dae</uri>
-          </mesh>
-        </geometry>
-      </visual>
-      <collision name="collision-base">
-        <pose>0 0 -0.0145 0 0 0</pose>
-        <geometry>
-          <box>
-            <size>0.05 0.05 0.041</size>
-          </box>
-        </geometry>
-      </collision>
-      <collision name="collision-top">
-        <pose>0 0 0.0205 0 0 0</pose>
-        <geometry>
-          <cylinder>
-            <radius>0.021</radius>
-            <length>0.029</length>
-          </cylinder>
-        </geometry>
-      </collision>
-      <sensor name="laser" type="gpu_ray">
-        <pose>0.01 0 0.0175 0 -0 0</pose>
-        <ray>
-          <scan>
-            <horizontal>
-              <samples>720</samples>
-              <resolution>1</resolution>
-              <min_angle>-1.57</min_angle>
-              <max_angle>1.57</max_angle>
-            </horizontal>
-          </scan>
-          <range>
-            <min>0.05</min>
-            <max>20</max>
-            <resolution>0.01</resolution>
-          </range>
-        </ray>
-        <noise>
-          <type>gaussian</type>
-          <mean>0.0</mean>
-          <stddev>0.005</stddev>
-        </noise>
-        <plugin name="gazebo_ros_head_hokuyo_controller" filename="libgazebo_ros_gpu_laser.so">
-          <topicName>/scan</topicName>
-          <frameName>laser</frameName>
-        </plugin>
-        <always_on>1</always_on>
-        <update_rate>40</update_rate>
-        <visualize>true</visualize>
-      </sensor>
-    </link>
-    <link name="cam_d1_link">
-      <pose>0.285 0.08 0.376 0 0 0</pose>
-      <inertial>
-        <mass>0.2</mass>
-        <inertia>
-          <ixx>0.014395</ixx>
-          <ixy>0</ixy>
-          <ixz>0</ixz>
-          <iyy>0.00384</iyy>
-          <iyz>0</iyz>
-          <izz>0.014136</izz>
-        </inertia>
-      </inertial>
-      <collision name="collision">
-        <geometry>
-          <box>
-            <size>0.008 0.13 0.02</size>
-          </box>
-        </geometry>
-      </collision>
-      <visual name="visual">
-        <geometry>
-          <mesh>
-            <uri>model://intel_realsense_r200/meshes/realsense_r200.dae</uri>
-          </mesh>
-        </geometry>
-      </visual>
-      <sensor name="imu_sensor" type="imu">
-        <gravity>true</gravity>
-        <always_on>true</always_on>
-        <update_rate>100</update_rate>
-        <visualize>true</visualize>
-        <plugin filename="libgazebo_ros_imu_sensor.so" name="imu_plugin">
-          <topicName>/cam_d1/imu</topicName>
-          <bodyName>cam_d1_link</bodyName>
-          <updateRateHZ>0.0</updateRateHZ>
-          <gaussianNoise>0.002</gaussianNoise>
-          <xyzOffset>0 0 0</xyzOffset>
-          <rpyOffset>0 0 0</rpyOffset>
-          <frameName>cam_d1_link</frameName>
-          <initialOrientationAsReference>false</initialOrientationAsReference>
-        </plugin>
-        <pose>0 0 0 0 0 0</pose>
-      </sensor>
-      <sensor name="camera" type="depth">
-        <!--pose>0.001 -0.045 0.003 0 0 0</pose-->
-        <pose> 0 0 0 0 0 0 </pose>
-        <visualize>true</visualize>
-        <update_rate>15</update_rate>
-        <camera>
-          <horizontal_fov>1.204</horizontal_fov>
-          <image>
-            <width>1280</width>
-            <height>720</height>
-            <format>R8G8B8</format>
-          </image>
-          <noise>
-            <type>gaussian</type>
-            <mean>0.0</mean>
-            <stddev>0.007</stddev>
-          </noise>
-        </camera>
-        <plugin name="camera_plugin" filename="libgazebo_ros_openni_kinect.so">
-          <baseline>0.2</baseline>
-          <alwaysOn>true</alwaysOn>
-          <!-- Keep this zero, update_rate in the parent <sensor> tag
-            will control the frame rate. -->
-          <updateRate>0.0</updateRate>
-          <cameraName>cam_d1</cameraName>
-          <imageTopicName>/cam_d1/color/image_raw</imageTopicName>
-          <cameraInfoTopicName>/cam_d1/color/camera_info</cameraInfoTopicName>
-          <depthImageTopicName>/cam_d1/depth/image_rect_raw</depthImageTopicName>
-          <depthImageCameraInfoTopicName>/cam_d1/depth/camera_info</depthImageCameraInfoTopicName>
-          <pointCloudTopicName>/cam_d1/depth/color/points</pointCloudTopicName>
-          <frameName>cam_d1_depth_link</frameName>
-          <pointCloudCutoff>0.3</pointCloudCutoff>
-          <pointCloudCutoffMax>8.0</pointCloudCutoffMax>
-          <distortionK1>0</distortionK1>
-          <distortionK2>0</distortionK2>
-          <distortionK3>0</distortionK3>
-          <distortionT1>0</distortionT1>
-          <distortionT2>0</distortionT2>
-          <CxPrime>0</CxPrime>
-          <Cx>0</Cx>
-          <Cy>0</Cy>
-          <focalLength>0</focalLength>
-          <hackBaseline>0</hackBaseline>
-        </plugin>
-      </sensor>
-    </link>
-    <link name="cam_d2_link">
-      <pose>-0.285 -0.08 0.376 0 0 3.14159</pose>
-      <inertial>
-        <mass>0.2</mass>
-        <inertia>
-          <ixx>0.014395</ixx>
-          <ixy>0</ixy>
-          <ixz>0</ixz>
-          <iyy>0.00384</iyy>
-          <iyz>0</iyz>
-          <izz>0.014136</izz>
-        </inertia>
-      </inertial>
-      <collision name="collision">
-        <geometry>
-          <box>
-            <size>0.008 0.13 0.02</size>
-          </box>
-        </geometry>
-      </collision>
-      <visual name="visual">
-        <geometry>
-          <mesh>
-            <uri>model://intel_realsense_r200/meshes/realsense_r200.dae</uri>
-          </mesh>
-        </geometry>
-      </visual>
-      <sensor name="imu_sensor" type="imu">
-        <always_on>true</always_on>
-        <update_rate>100</update_rate>
-        <visualize>true</visualize>
-        <gravity>true</gravity>
-        <plugin filename="libgazebo_ros_imu_sensor.so" name="imu_plugin">
-          <topicName>/cam_d2/imu</topicName>
-          <bodyName>cam_d2_link</bodyName>
-          <updateRateHZ>0.0</updateRateHZ>
-          <gaussianNoise>0.002</gaussianNoise>
-          <xyzOffset>0 0 0</xyzOffset>
-          <rpyOffset>0 0 0</rpyOffset>
-          <frameName>cam_d2_link</frameName>
-          <initialOrientationAsReference>false</initialOrientationAsReference>
-        </plugin>
-        <pose>0 0 0 0 0 0</pose>
-      </sensor>
-      <sensor name="camera" type="depth">
-        <!--pose>0.001 -0.045 0.003 0 0 0</pose-->
-        <pose> 0 0 0 0 0 0 </pose>
-        <visualize>true</visualize>
-        <update_rate>15</update_rate>
-        <camera>
-          <horizontal_fov>1.204</horizontal_fov>
-          <image>
-            <width>1280</width>
-            <height>720</height>
-            <format>R8G8B8</format>
-          </image>
-          <noise>
-            <type>gaussian</type>
-            <mean>0.0</mean>
-            <stddev>0.007</stddev>
-          </noise>
-        </camera>
-        <plugin name="camera_plugin" filename="libgazebo_ros_openni_kinect.so">
-          <baseline>0.2</baseline>
-          <alwaysOn>true</alwaysOn>
-          <!-- Keep this zero, update_rate in the parent <sensor> tag
-            will control the frame rate. -->
-          <updateRate>0.0</updateRate>
-          <cameraName>cam_d2</cameraName>
-          <imageTopicName>/cam_d2/color/image_raw</imageTopicName>
-          <cameraInfoTopicName>/cam_d2/color/camera_info</cameraInfoTopicName>
-          <depthImageTopicName>/cam_d2/depth/image_rect_raw</depthImageTopicName>
-          <depthImageCameraInfoTopicName>/cam_d2/depth/camera_info</depthImageCameraInfoTopicName>
-          <pointCloudTopicName>/cam_d2/depth/color/points</pointCloudTopicName>
-          <frameName>cam_d2_depth_link</frameName>
-          <pointCloudCutoff>0.3</pointCloudCutoff>
-          <pointCloudCutoffMax>6.0</pointCloudCutoffMax>
-          <distortionK1>0</distortionK1>
-          <distortionK2>0</distortionK2>
-          <distortionK3>0</distortionK3>
-          <distortionT1>0</distortionT1>
-          <distortionT2>0</distortionT2>
-          <CxPrime>0</CxPrime>
-          <Cx>0</Cx>
-          <Cy>0</Cy>
-          <focalLength>0</focalLength>
-          <hackBaseline>0</hackBaseline>
-        </plugin>
-      </sensor>
     </link>
     <!-- Powerd Caster steering joints -->
@@ -700,17 +441,280 @@
       </axis>
     </joint>
-    <joint name="hokuyo_joint" type="fixed">
-      <child>hokuyo</child>
-      <parent>base_link</parent>
-    </joint>
-    <joint name="front_rs_joint" type="fixed">
-      <child>cam_d1_link</child>
-      <parent>base_link</parent>
-    </joint>
-    <joint name="rear_rs_joint" type="fixed">
-      <child>cam_d2_link</child>
-      <parent>base_link</parent>
-    </joint>
+  </gazebo>
+  <gazebo reference="laser">
+      <inertial>
+        <mass>0.1</mass>
+        <inertia>
+          <ixx>0.01</ixx>
+          <ixy>0</ixy>
+          <ixz>0</ixz>
+          <iyy>0.01</iyy>
+          <iyz>0</iyz>
+          <izz>0.01</izz>
+        </inertia>
+      </inertial>
+      <visual name="visual">
+        <pose>0 0 -0.0175 0 0 0</pose>
+        <geometry>
+          <mesh>
+            <uri>model://hokuyo/meshes/hokuyo.dae</uri>
+          </mesh>
+        </geometry>
+      </visual>
+      <collision name="collision-base">
+        <pose>0 0 -0.032 0 0 0</pose>
+        <geometry>
+          <box>
+            <size>0.05 0.05 0.041</size>
+          </box>
+        </geometry>
+      </collision>
+      <collision name="collision-top">
+        <pose>0 0 0.003 0 0 0</pose>
+        <geometry>
+          <cylinder>
+            <radius>0.021</radius>
+            <length>0.029</length>
+          </cylinder>
+        </geometry>
+      </collision>
+      <sensor name="laser" type="gpu_ray">
+        <pose>0.01 0 0 0 -0 0</pose>
+        <ray>
+          <scan>
+            <horizontal>
+              <samples>720</samples>
+              <resolution>1</resolution>
+              <min_angle>-1.57</min_angle>
+              <max_angle>1.57</max_angle>
+            </horizontal>
+          </scan>
+          <range>
+            <min>0.05</min>
+            <max>20</max>
+            <resolution>0.01</resolution>
+          </range>
+        </ray>
+        <noise>
+          <type>gaussian</type>
+          <mean>0.0</mean>
+          <stddev>0.005</stddev>
+        </noise>
+        <plugin name="gazebo_ros_head_hokuyo_controller" filename="libgazebo_ros_gpu_laser.so">
+          <topicName>scan</topicName>
+          <frameName>laser</frameName>
+        </plugin>
+        <always_on>1</always_on>
+        <update_rate>40</update_rate>
+        <visualize>true</visualize>
+      </sensor>
+  </gazebo>
+  <gazebo name="cam_d1_link">
+      <inertial>
+        <mass>0.2</mass>
+        <inertia>
+          <ixx>0.014395</ixx>
+          <ixy>0</ixy>
+          <ixz>0</ixz>
+          <iyy>0.00384</iyy>
+          <iyz>0</iyz>
+          <izz>0.014136</izz>
+        </inertia>
+      </inertial>
+      <collision name="collision">
+        <geometry>
+          <box>
+            <size>0.008 0.13 0.02</size>
+          </box>
+        </geometry>
+      </collision>
+      <visual name="visual">
+        <geometry>
+          <mesh>
+            <uri>model://intel_realsense_r200/meshes/realsense_r200.dae</uri>
+          </mesh>
+        </geometry>
+      </visual>
+      <sensor name="imu_sensor" type="imu">
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